Commit message: update

File: src/xxx_description/urdf/xxx.xacro (robot description, xacro)
@@ -6,5 +6,5 @@
     <xacro:include filename="$(find xxx_description)/urdf/xxx_castor.xacro"/>
     <xacro:include filename="$(find xxx_description)/urdf/xxx_sensor.xacro"/>
-    <!-- <xacro:include filename="$(find xxx_description)/urdf/xxx_gazebo.xacro"/> -->
+    <xacro:include filename="$(find xxx_description)/urdf/xxx_gazebo.xacro"/>
     <xacro:chassis/>
     <xacro:wheel
@@ -57,4 +57,4 @@
         parent="base_link"/>
     <xacro:sensor />
-    <!-- <gazebo />   -->
+    <gazebo/>
 </robot>

File: src/xxx_description/urdf/xxx_gazebo.xacro (robot description, xacro)
@@ -1,5 +1,25 @@
 <?xml version="1.0"?>
 <robot name="xxx_gazebo"  xmlns:xacro="http://ros.org/wiki/xacro">
-    <xacro:macro name="gazebo" params="">
+<!-- <xacro:macro name="gazebo" params=""> -->
+    <gazebo>
+    <plugin name="differential_drive_controller" filename="libgazebo_ros_diff_drive.so">
+      <alwaysOn>true</alwaysOn>
+      <updateRate>20</updateRate>
+      <left_joint>left_wheel_joint</left_joint>
+      <right_joint>right_wheel_joint</right_joint>
+      <wheel_separation>0.4</wheel_separation>
+      <wheel_diameter>0.1</wheel_diameter>
+      <max_wheel_torque>20</max_wheel_torque>
+      <max_wheel_acceleration>1.0</max_wheel_acceleration>
+      <command_topic>cmd_vel</command_topic>
+      <command_topic>odom</command_topic>
+      <publish_odom>true</publish_odom>
+      <publish_odom_tf>false</publish_odom_tf>
+      <publish_wheel_tf>true</publish_wheel_tf>
+      <odometry_topic>odom</odometry_topic>
+      <odometry_frame>odom</odometry_frame>
+      <robot_base_frame>base_footprint</robot_base_frame>
+    </plugin>
+    </gazebo>
     <!-- CHASIS -->
     <gazebo reference="base_link">
@@ -22,6 +42,6 @@
     <!-- WHEEL -->
     <gazebo>
-        <plugin name="gazebo_ros_control" filename="libgazebo_ros_control.so">
-            <robotNamespace>xxx</robotNamespace>
+        <plugin name="gazebo-ros2-control" filename="gazebo_ros2_control">
+            <robotNamespace>coconut</robotNamespace>
         </plugin>
     </gazebo>
@@ -36,5 +56,5 @@
         <material>Gazebo/Black</material>
     </gazebo>
-    <!-- CASTER -->
+     <!-- CASTER -->
     <gazebo reference="right_front_castor">
         <mu1>0.1</mu1>
@@ -57,102 +77,11 @@
         <material>Gazebo/Yellow</material>
     </gazebo>
-    <!-- LIDAR -->
+     <!-- LIDAR -->
     <gazebo reference="lidar">
-        <material>Gazebo/Blue</material>
+        <material>Gazebo/Red</material>
     </gazebo>
-    <gazebo reference="lidar">
-    <sensor type="ray" name="lidar_plugin">
-        <pose>0 0 0 0 0 0</pose>
-        <visualize>true</visualize>
-        <update_rate>7</update_rate>
-        <ray>
-        <scan>
-            <horizontal>
-            <samples>720</samples>
-            <resolution>1</resolution>
-            <min_angle>0</min_angle>
-            <max_angle>6.28319</max_angle>
-            </horizontal>
-        </scan>
-        <range>
-            <min>0.05</min>
-            <max>16</max>
-            <!-- <resolution>0.015</resolution> -->
-            <resolution>0.03</resolution>
-        </range>
-        <noise>
-            <type>gaussian</type>
-            <mean>0.0</mean>
-            <!-- <stddev>0.02</stddev> -->
-            <stddev>0.03</stddev>
-        </noise>
-        </ray>
-        <plugin name="gazebo_ros_lidar" filename="libgazebo_ros_laser.so">
-        <topicName>scan</topicName>
-        <frameName>lidar</frameName>
-        </plugin>
-    </sensor>
-  </gazebo>
-    <!-- CAMERA -->
+     <!-- CAMERA -->
     <gazebo reference="t265">
-        <material>Gazebo/Blue</material>
-    </gazebo>
-    <gazebo reference="camera">
-        <sensor type="camera" name="camera1">
-          <update_rate>30.0</update_rate>
-          <camera name="head">
-            <horizontal_fov>1.3962634</horizontal_fov>
-            <image>
-              <width>640</width>
-              <height>360</height>
-              <format>R8G8B8</format>
-            </image>
-            <clip>
-              <near>0.02</near>
-              <far>300</far>
-            </clip>
-            <lens>
-                <intrinsics>
-                  <fx>381.36246688113556</fx>
-                  <fy>381.36246688113556</fy>
-                  <cx>320.5</cx>
-                  <cy>180.5</cy>
-                  <s>0</s>
-                </intrinsics>
-            </lens>
-            <noise>
-              <type>gaussian</type>
-              <!-- Noise is sampled independently per pixel on each frame.
-                   That pixel's noise value is added to each of its color
-                   channels, which at that point lie in the range [0,1]. -->
-              <mean>0.0</mean>
-              <stddev>0.000001</stddev>
-            </noise>
-          </camera>
-          <plugin name="camera_controller" filename="libgazebo_ros_camera.so">
-            <alwaysOn>true</alwaysOn>
-            <updateRate>0.0</updateRate>
-            <cameraName>camera</cameraName>
-            <imageTopicName>image_raw</imageTopicName>
-            <cameraInfoTopicName>camera_info</cameraInfoTopicName>
-            <frameName>camera_optical</frameName>
-            <hackBaseline>0.07</hackBaseline>
-            <distortionK1>0.0</distortionK1>
-            <distortionK2>0.0</distortionK2>
-            <distortionK3>0.0</distortionK3>
-            <distortionT1>0.0</distortionT1>
-            <distortionT2>0.0</distortionT2>
-          </plugin>
-        </sensor>
-    </gazebo>
-    <gazebo>
-        <plugin name="imu_plugin" filename="libgazebo_ros_imu.so">
-          <alwaysOn>true</alwaysOn>
-          <bodyName>base_footprint</bodyName>
-          <topicName>imu</topicName>
-          <serviceName>imu_service</serviceName>
-          <gaussianNoise>0.0</gaussianNoise>
-          <updateRate>20.0</updateRate>
-        </plugin>
+        <material>Gazebo/Green</material>
     </gazebo>
     <!-- ULTRASONIC -->
@@ -181,4 +110,14 @@
         <material>Gazebo/Blue</material>
     </gazebo>
-</xacro:macro>
+    <!-- <gazebo>
+        <plugin name="imu_plugin" filename="libgazebo_ros_imu.so">
+          <alwaysOn>true</alwaysOn>
+          <bodyName>base_footprint</bodyName>
+          <topicName>imu</topicName>
+          <serviceName>imu_service</serviceName>
+          <gaussianNoise>0.0</gaussianNoise>
+          <updateRate>20.0</updateRate>
+        </plugin>
+    </gazebo> -->
+<!-- </xacro:macro> -->
 </robot>
